File: _autosave-Lessisbore-pcb.sch (KiCad schematic (older format))
At the start: 24 parts, among them SW1 SW_Push, U1 ATmega32U4-AU, Y1 16Mhz

Commit message: Termino de preparar pcb
Parts:
- renumbered R3 to R1, R1 to R3
Changed lines of the file:
@@
 Wire Wire Line
 	1800 3400 1950 3400
-$Comp
-L Device:R_Small R1
-U 1 1 608B2D96
-P 2050 3400
-F 0 "R1" V 1854 3400 50  0000 C CNN
-F 1 "22" V 1945 3400 50  0000 C CNN
-F 2 "Resistor_SMD:R_0805_2012Metric" H 2050 3400 50  0001 C CNN
-F 3 "~" H 2050 3400 50  0001 C CNN
-	1    2050 3400
-	0    1    1    0
-$EndComp
 Wire Wire Line
 	4900 4400 5100 4400
@@
 	2900 2300 2600 2300
 $Comp
-L Device:R_Small R3
+L Device:R_Small R1
 U 1 1 6091BF7D
 P 2900 2000
-F 0 "R3" H 2959 2046 50  0000 L CNN
+F 0 "R1" H 2959 2046 50  0000 L CNN
 F 1 "10k" H 2959 1955 50  0000 L CNN
 F 2 "Resistor_SMD:R_0805_2012Metric" H 2900 2000 50  0001 C CNN
@@
 Wire Wire Line
 	2250 2800 2450 2800
+$Comp
+L Device:R_Small R3
+U 1 1 608B2D96
+P 2050 3400
+F 0 "R3" V 1854 3400 50  0000 C CNN
+F 1 "22" V 1945 3400 50  0000 C CNN
+F 2 "Resistor_SMD:R_0805_2012Metric" H 2050 3400 50  0001 C CNN
+F 3 "~" H 2050 3400 50  0001 C CNN
+	1    2050 3400
+	0    1    1    0
+$EndComp
 $EndSCHEMATC
