File: Lessisbore-pcb.sch (KiCad schematic (older format))
At the start: 24 parts, among them SW1 SW_Push, U1 ATmega32U4-AU, Y1 16Mhz

Commit message: Refill
Parts:
- renumbered C3 to C1, C4 to C2, C6 to C3, C1 to C4, C2 to C5, C5 to C6, D3 to D2, D2 to D3, MX3 to MX2, MX2 to MX3, R3 to R1, R1 to R3
Connections:
- net COL0: now also U1.29 (PB5)
- net COL1: now also U1.28 (PB4)
- net GND: now also USB1.6 (SHIELD)
- net ROW0: now also U1.27 (PD7)
- net ROW1: now also U1.30 (PB6)
Changed lines of the file:
@@
 Comment4 ""
 $EndDescr
-$Comp
-L random-keyboard-parts:Molex-0548190589 USB1
-U 1 1 6091F629
-P 6375 2300
-F 0 "USB1" V 6912 2267 60  0000 C CNN
-F 1 "Molex-0548190589" V 6806 2267 60  0000 C CNN
-F 2 "random-keyboard-parts:Molex-0548190589" H 6375 2300 60  0001 C CNN
-F 3 "" H 6375 2300 60  0001 C CNN
-	1    6375 2300
-	0    -1   -1   0
-$EndComp
 Text GLabel 6675 2200 2    50   Input ~ 0
 D-
@@
 	7025 2100 7275 2100
 Wire Wire Line
-	6675 2500 6825 2500
-$Comp
-L power:GND #PWR0103
-U 1 1 60931900
-P 6825 2500
-F 0 "#PWR0103" H 6825 2250 50  0001 C CNN
-F 1 "GND" H 6830 2327 50  0000 C CNN
-F 2 "" H 6825 2500 50  0001 C CNN
-F 3 "" H 6825 2500 50  0001 C CNN
-	1    6825 2500
-	1    0    0    -1
-$EndComp
-Wire Wire Line
 	7125 4800 7025 4800
 Wire Wire Line
@@
 $EndComp
 $Comp
-L MX_Alps_Hybrid:MX-NoLED MX2
+L MX_Alps_Hybrid:MX-NoLED MX3
 U 1 1 60932393
 P 7175 4650
-F 0 "MX2" H 7208 4873 60  0000 C CNN
+F 0 "MX3" H 7208 4873 60  0000 C CNN
 F 1 "MX-NoLED" H 7208 4799 20  0000 C CNN
 F 2 "MX_Alps_Hybrid:MX-1U" H 6550 4625 60  0001 C CNN
@@
 	7925 4000 7825 4000
 $Comp
-L MX_Alps_Hybrid:MX-NoLED MX3
+L MX_Alps_Hybrid:MX-NoLED MX2
 U 1 1 60958F68
 P 7975 3850
-F 0 "MX3" H 8008 4073 60  0000 C CNN
+F 0 "MX2" H 8008 4073 60  0000 C CNN
 F 1 "MX-NoLED" H 8008 3999 20  0000 C CNN
 F 2 "MX_Alps_Hybrid:MX-1U" H 7350 3825 60  0001 C CNN
@@
 $EndComp
 $Comp
-L Device:D_Small D3
+L Device:D_Small D2
 U 1 1 6097465A
 P 7825 4100
-F 0 "D3" H 7915 4161 50  0000 L CNN
+F 0 "D2" H 7915 4161 50  0000 L CNN
 F 1 "SOD-123" H 8073 4161 50  0000 L CNN
 F 2 "Diode_SMD:D_SOD-123" V 7825 4100 50  0001 C CNN
@@
 $EndComp
 $Comp
-L Device:D_Small D2
+L Device:D_Small D3
 U 1 1 60976C6C
 P 7025 4900
-F 0 "D2" H 7115 4961 50  0000 L CNN
+F 0 "D3" H 7115 4961 50  0000 L CNN
 F 1 "SOD-123" H 7273 4961 50  0000 L CNN
 F 2 "Diode_SMD:D_SOD-123" V 7025 4900 50  0001 C CNN
@@
 COL1
 $Comp
-L Device:C_Small C1
+L Device:C_Small C4
 U 1 1 608FF7BF
 P 1200 4875
-F 0 "C1" H 1292 4921 50  0000 L CNN
+F 0 "C4" H 1292 4921 50  0000 L CNN
 F 1 "0.1uF" H 1292 4830 50  0000 L CNN
 F 2 "Capacitor_SMD:C_0805_2012Metric" H 1200 4875 50  0001 C CNN
@@
 Wire Wire Line
 	1800 3400 1950 3400
-$Comp
-L Device:R_Small R1
-U 1 1 608B2D96
-P 2050 3400
-F 0 "R1" V 1854 3400 50  0000 C CNN
-F 1 "22" V 1945 3400 50  0000 C CNN
-F 2 "Resistor_SMD:R_0805_2012Metric" H 2050 3400 50  0001 C CNN
-F 3 "~" H 2050 3400 50  0001 C CNN
-	1    2050 3400
-	0    1    1    0
-$EndComp
 Wire Wire Line
 	4900 4400 5100 4400
@@
 	2500 3300 3000 3300
 $Comp
-L Device:C_Small C6
+L Device:C_Small C3
 U 1 1 608ED982
 P 2400 3700
-F 0 "C6" H 2492 3746 50  0000 L CNN
+F 0 "C3" H 2492 3746 50  0000 L CNN
 F 1 "1uF" H 2492 3655 50  0000 L CNN
 F 2 "Capacitor_SMD:C_0805_2012Metric" H 2400 3700 50  0001 C CNN
@@
 $EndComp
 $Comp
-L Device:C_Small C5
+L Device:C_Small C6
 U 1 1 608F9E34
 P 2250 4875
-F 0 "C5" H 2342 4921 50  0000 L CNN
+F 0 "C6" H 2342 4921 50  0000 L CNN
 F 1 "0.1uF" H 2342 4830 50  0000 L CNN
 F 2 "Capacitor_SMD:C_0805_2012Metric" H 2250 4875 50  0001 C CNN
@@
 $EndComp
 $Comp
-L Device:C_Small C2
+L Device:C_Small C5
 U 1 1 608FE427
 P 1700 4875
-F 0 "C2" H 1792 4921 50  0000 L CNN
+F 0 "C5" H 1792 4921 50  0000 L CNN
 F 1 "0.1uF" H 1792 4830 50  0000 L CNN
 F 2 "Capacitor_SMD:C_0805_2012Metric" H 1700 4875 50  0001 C CNN
@@
 $EndComp
 $Comp
-L Device:C_Small C3
+L Device:C_Small C1
 U 1 1 6090AD00
 P 1750 2350
-F 0 "C3" V 1521 2350 50  0000 C CNN
+F 0 "C1" V 1521 2350 50  0000 C CNN
 F 1 "22pF" V 1612 2350 50  0000 C CNN
 F 2 "Capacitor_SMD:C_0805_2012Metric" H 1750 2350 50  0001 C CNN
@@
 $EndComp
 $Comp
-L Device:C_Small C4
+L Device:C_Small C2
 U 1 1 6090C049
 P 1750 2800
-F 0 "C4" V 1521 2800 50  0000 C CNN
+F 0 "C2" V 1521 2800 50  0000 C CNN
 F 1 "22pF" V 1612 2800 50  0000 C CNN
 F 2 "Capacitor_SMD:C_0805_2012Metric" H 1750 2800 50  0001 C CNN
@@
 	2900 2300 2600 2300
 $Comp
-L Device:R_Small R3
+L Device:R_Small R1
 U 1 1 6091BF7D
 P 2900 2000
-F 0 "R3" H 2959 2046 50  0000 L CNN
+F 0 "R1" H 2959 2046 50  0000 L CNN
 F 1 "10k" H 2959 1955 50  0000 L CNN
 F 2 "Resistor_SMD:R_0805_2012Metric" H 2900 2000 50  0001 C CNN
@@
 Wire Wire Line
 	2250 2800 2450 2800
+$Comp
+L Device:R_Small R3
+U 1 1 608B2D96
+P 2050 3400
+F 0 "R3" V 1854 3400 50  0000 C CNN
+F 1 "22" V 1945 3400 50  0000 C CNN
+F 2 "Resistor_SMD:R_0805_2012Metric" H 2050 3400 50  0001 C CNN
+F 3 "~" H 2050 3400 50  0001 C CNN
+	1    2050 3400
+	0    1    1    0
+$EndComp
+Text GLabel 4200 4200 2    50   Input ~ 0
+ROW0
+Text GLabel 4200 2800 2    50   Input ~ 0
+COL0
+Text GLabel 4200 2900 2    50   Input ~ 0
+ROW1
+Text GLabel 4200 2700 2    50   Input ~ 0
+COL1
+$Comp
+L random-keyboard-parts:Molex-0548190589 USB1
+U 1 1 6091F629
+P 6375 2300
+F 0 "USB1" V 6912 2267 60  0000 C CNN
+F 1 "Molex-0548190589" V 6806 2267 60  0000 C CNN
+F 2 "random-keyboard-parts:Molex-0548190589" H 6375 2300 60  0001 C CNN
+F 3 "" H 6375 2300 60  0001 C CNN
+	1    6375 2300
+	0    -1   -1   0
+$EndComp
+Wire Wire Line
+	6675 2000 6775 2000
+$Comp
+L power:GND #PWR?
+U 1 1 60A65E66
+P 7000 2500
+F 0 "#PWR?" H 7000 2250 50  0001 C CNN
+F 1 "GND" H 7005 2327 50  0000 C CNN
+F 2 "" H 7000 2500 50  0001 C CNN
+F 3 "" H 7000 2500 50  0001 C CNN
+	1    7000 2500
+	1    0    0    -1
+$EndComp
+Wire Wire Line
+	6775 2000 6775 2500
+Wire Wire Line
+	6675 2500 6775 2500
+Connection ~ 6775 2500
+Wire Wire Line
+	6775 2500 7000 2500
 $EndSCHEMATC
