File: _autosave-Lessisbore-pcb.kicad_pcb (KiCad board)
At the start: 2 copper layers, 78.6 x 38.1 mm, 24 parts, among them SW1 SW_Push, U1 ATmega32U4-AU, Y1 16Mhz

Commit message: Refill
Parts:
- D1, D2, D3, D4: moved to B.Cu
- moved C7 6.41 mm to (33.0, 50.0), turned to 270 degrees
- moved F1 2.70 mm to (18.2, 42.3), turned to 90 degrees
- moved R2 2.00 mm to (23.7, 35.9)
- moved SW1 1.99 mm to (21.0, 57.5)
- moved R3 1.81 mm to (20.6, 35.9)
- moved C4 0.67 mm to (35.1, 37.3)
- moved C3 0.61 mm to (32.3, 44.7)
- moved R1 0.25 mm to (31.5, 37.3), turned to 270 degrees
- moved USB1 0.25 mm to (23.0, 25.7)
Connections:
- U1 pad 27: Net-(U1-Pad27) -> ROW0
- U1 pad 28: Net-(U1-Pad28) -> COL1
- U1 pad 29: Net-(U1-Pad29) -> COL0
- U1 pad 30: Net-(U1-Pad30) -> ROW1
- USB1 pad 6: Net-(USB1-Pad6) -> GND
Routing:
- net GND: track 0.00 -> 153.5 mm
- net +5V: track 0.00 -> 100.7 mm, vias 0 -> 5
- net COL1: track 0.00 -> 51.8 mm
- net ROW1: track 0.00 -> 50.7 mm
- net ROW0: track 0.00 -> 49.3 mm
- net Net-(R1-Pad2): track 0.00 -> 33.1 mm, vias 0 -> 2
- net COL0: track 0.00 -> 32.4 mm
- net Net-(R3-Pad1): track 0.00 -> 24.2 mm
- net Net-(R2-Pad1): track 0.00 -> 23.1 mm
- net VCC: track 0.00 -> 12.8 mm
- net Net-(C2-Pad1): track 0.00 -> 12.6 mm
- net Net-(C1-Pad1): track 0.00 -> 10.3 mm
- net Net-(D2-Pad2): track 0.00 -> 7.82 mm
- net Net-(D1-Pad2): track 0.00 -> 7.33 mm
- net Net-(D3-Pad2): track 0.00 -> 6.82 mm
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- added copper zone on B.Cu, net GND
Other:
- outline, holes or cut-outs redrawn
- net class Power added: clearance 0.2, trace_width 0.381, via_dia 0.8, via_drill 0.4
- rule trace_min: 0.2 -> 0
